File: PCB/CAMERA_SHIELD.sch (EAGLE design)
At the start: 72 parts, among them IC4 LSF0204PWR, J1 47346-0001, Q1 FDN304P, Q2 FDN304P, Q3 SSM3J338R,LF, Q4 SSM3J338R,LF, U1 LARA-R2

Commit message: new route
Connections:
- removed net RX: IC4.A2, RXD.TP
- removed net TX: IC4.A1, TXD.TP
- new net N$11: RTS.TP
- new net N$13: RXD.TP
- new net N$4: CTS.TP
- net CTS: now also IC4.A1; no longer CTS.TP, IC4.A3
- net RTS: now also IC4.A2; no longer IC4.A4, RTS.TP
- net RXD: now also IC4.A4
- net TXD: now also IC4.A3, TXD.TP
Changed lines of the file:
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@@
-</segment>
-</bus>
-<bus name="UART:CTS,RTS,RX,TX">
-<segment>
-<wire x1="43.95" y1="279.39" x2="43.95" y2="292.09" width="0.762" layer="92"/>
-</segment>
-</bus>
-<bus name="B$1">
-<segment>
-<wire x1="43.79" y1="291.15" x2="43.79" y2="292.33" width="0.762" layer="92"/>
-<wire x1="43.79" y1="292.33" x2="100.24" y2="292.33" width="0.762" layer="92"/>
 </segment>
 </bus>
@@
 <net name="RTS" class="0">
 <segment>
-<pinref part="IC4" gate="G$1" pin="A4"/>
-<wire x1="38.87" y1="281.93" x2="43.95" y2="281.93" width="0.1524" layer="91"/>
-</segment>
-<segment>
-<pinref part="RTS" gate="G$1" pin="TP"/>
-<wire x1="64.27" y1="292.09" x2="64.27" y2="297.17" width="0.1524" layer="91"/>
-</segment>
-<segment>
 <pinref part="U1" gate="G$1" pin="RTS"/>
 <wire x1="132.99" y1="257.25" x2="116.87" y2="257.25" width="0.1524" layer="91"/>
@@
 <label x="119.43" y="257.15" size="1.778" layer="95"/>
 </segment>
+<segment>
+<pinref part="IC4" gate="G$1" pin="A2"/>
+<wire x1="38.87" y1="287.01" x2="43.63" y2="287.01" width="0.1524" layer="91"/>
+<wire x1="43.63" y1="287.01" x2="43.63" y2="286.88" width="0.1524" layer="91"/>
+<label x="39.74" y="286.8" size="1.778" layer="95"/>
+</segment>
 </net>
 <net name="CTS" class="0">
-<segment>
-<pinref part="IC4" gate="G$1" pin="A3"/>
-<wire x1="38.87" y1="284.47" x2="43.95" y2="284.47" width="0.1524" layer="91"/>
-</segment>
-<segment>
-<pinref part="CTS" gate="G$1" pin="TP"/>
-<wire x1="54.11" y1="292.09" x2="54.11" y2="297.17" width="0.1524" layer="91"/>
-</segment>
 <segment>
 <pinref part="U1" gate="G$1" pin="CTS"/>
@@
 <label x="119.16" y="254.55" size="1.778" layer="95"/>
 </segment>
-</net>
-<net name="TX" class="0">
 <segment>
 <pinref part="IC4" gate="G$1" pin="A1"/>
 <wire x1="38.87" y1="289.55" x2="43.95" y2="289.55" width="0.1524" layer="91"/>
-</segment>
-<segment>
-<pinref part="TXD" gate="G$1" pin="TP"/>
-<wire x1="74.43" y1="292.09" x2="74.43" y2="297.17" width="0.1524" layer="91"/>
-</segment>
-</net>
-<net name="RX" class="0">
-<segment>
-<pinref part="IC4" gate="G$1" pin="A2"/>
-<wire x1="38.87" y1="287.01" x2="43.95" y2="287.01" width="0.1524" layer="91"/>
-</segment>
-<segment>
-<pinref part="RXD" gate="G$1" pin="TP"/>
-<wire x1="84.59" y1="292.09" x2="84.59" y2="297.17" width="0.1524" layer="91"/>
+<label x="39.45" y="289.64" size="1.778" layer="95"/>
 </segment>
 </net>
@@
 <label x="119.88" y="262.32" size="1.778" layer="95"/>
 </segment>
+<segment>
+<pinref part="IC4" gate="G$1" pin="A3"/>
+<wire x1="38.87" y1="284.47" x2="43.74" y2="284.47" width="0.1524" layer="91"/>
+<label x="39.54" y="284.43" size="1.778" layer="95"/>
+<pinref part="TXD" gate="G$1" pin="TP"/>
+<wire x1="74.43" y1="297.17" x2="74.43" y2="284.47" width="0.1524" layer="91"/>
+<wire x1="74.43" y1="284.47" x2="43.75" y2="284.47" width="0.1524" layer="91"/>
+<wire x1="43.75" y1="284.47" x2="43.74" y2="284.47" width="0.1524" layer="91"/>
+<wire x1="43.74" y1="284.47" x2="43.74" y2="284.54" width="0.1524" layer="91"/>
+</segment>
 </net>
 <net name="RXD" class="0">
@@
 <wire x1="132.99" y1="259.79" x2="117.26" y2="259.79" width="0.1524" layer="91"/>
 <label x="119.57" y="259.62" size="1.778" layer="95"/>
+</segment>
+<segment>
+<pinref part="IC4" gate="G$1" pin="A4"/>
+<wire x1="38.87" y1="281.93" x2="43.95" y2="281.93" width="0.1524" layer="91"/>
+<label x="39.35" y="281.87" size="1.778" layer="95"/>
 </segment>
 </net>
@@
 </segment>
 </net>
+<net name="N$4" class="0">
+<segment>
+<pinref part="CTS" gate="G$1" pin="TP"/>
+<wire x1="54.11" y1="297.17" x2="54.11" y2="289.57" width="0.1524" layer="91"/>
+<wire x1="54.11" y1="289.57" x2="43.76" y2="289.57" width="0.1524" layer="91"/>
+</segment>
+</net>
+<net name="N$11" class="0">
+<segment>
+<pinref part="RTS" gate="G$1" pin="TP"/>
+<wire x1="64.27" y1="297.17" x2="64.27" y2="287.02" width="0.1524" layer="91"/>
+<wire x1="64.27" y1="287.02" x2="43.47" y2="287.02" width="0.1524" layer="91"/>
+</segment>
+</net>
+<net name="N$13" class="0">
+<segment>
+<pinref part="RXD" gate="G$1" pin="TP"/>
+<wire x1="84.59" y1="297.17" x2="84.59" y2="281.96" width="0.1524" layer="91"/>
+<wire x1="84.59" y1="281.96" x2="43.79" y2="281.96" width="0.1524" layer="91"/>
+</segment>
+</net>

Commit message: route gsm
Connections:
- removed net N$11: RTS.TP
- removed net N$13: RXD.TP
- removed net N$3: SDCARD.C1_VCC
- removed net N$4: CTS.TP
- removed net N$5: SDCARD.C3_CLK
- removed net N$6: SDCARD.C2_RST
- removed net N$8: SDCARD.C5_GND
- removed net N$9: SDCARD.C7_I/O
- removed net SIGNAL_C1: C7.1, TVS4.2
- removed net SIGNAL_C2: C8.1, TVS3.2
- removed net SIGNAL_C3: C9.1, TVS2.2
- removed net SIGNAL_C7: C10.1, TVS1.2
- removed net VIN: U1.V_INT
- net CTS: now also CTS.TP
- net RTS: now also RTS.TP
- net RXD: now also RXD.TP
- net SIM_CLK: now also C9.1, SDCARD.C3_CLK, TVS2.2
- net SIM_IO: now also C10.1, SDCARD.C7_I/O, TVS1.2
- net SIM_RST: now also C8.1, SDCARD.C2_RST, TVS3.2
- net VSIM: now also C7.1, SDCARD.C1_VCC, TVS4.2
- net V_INT: now also U1.V_INT

Commit message: stm32f7 with gsm-modul
Parts:
- added Q5: FDN304P, FDN304P:FDN304P
Connections:
- removed net PIR_IN: HUNG.PG12
- new net 3V3_SDCARD: Q5.D, SDCARD.T4_VDD
- net 3V3: now also HUNG.VDD_6, HUNG.V_DDSDMMC, Q5.S; no longer SDCARD.T4_VDD
- net MOSFET_SDCARD: now also Q5.G
- net PIR_INT: now also HUNG.PG12
- net VDD: no longer HUNG.VDD_6, HUNG.V_DDSDMMC

Commit message: smartcamera with gsm
Connections:
- new net N$196: U1.VCC
- net V_GSM: no longer U1.VCC
Changed lines of the file:
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@@
 <net name="V_GSM" class="0">
+<segment>
+<junction x="223.73" y="282.65"/>
+<wire x1="223.73" y1="277.57" x2="223.73" y2="282.65" width="0.1524" layer="91"/>
+<pinref part="C24" gate="G$1" pin="1"/>
+</segment>
 <segment>
 <wire x1="223.8" y1="282.65" x2="233.89" y2="282.65" width="0.1524" layer="91"/>
@@
 <wire x1="254.21" y1="282.65" x2="264.37" y2="282.65" width="0.1524" layer="91"/>
 <wire x1="274.53" y1="282.65" x2="287.23" y2="282.65" width="0.1524" layer="91"/>
-<wire x1="223.73" y1="277.57" x2="223.73" y2="282.65" width="0.1524" layer="91"/>
-<junction x="223.73" y="282.65"/>
 <wire x1="233.89" y1="277.57" x2="233.89" y2="282.65" width="0.1524" layer="91"/>
 <junction x="233.89" y="282.65"/>
@@
 <pinref part="C15" gate="G$1" pin="1"/>
 <pinref part="C17" gate="G$1" pin="1"/>
-<pinref part="C24" gate="G$1" pin="1"/>
 <pinref part="V_GSM" gate="G$1" pin="TP"/>
 <pinref part="TVS8" gate="G$1" pin="2"/>
-<pinref part="U1" gate="G$1" pin="VCC"/>
-<wire x1="178.71" y1="282.65" x2="223.75" y2="282.65" width="0.1524" layer="91"/>
 <wire x1="223.8" y1="282.55" x2="223.8" y2="282.65" width="0.1524" layer="91"/>
-<wire x1="223.75" y1="282.65" x2="223.95" y2="282.65" width="0.1524" layer="91"/>
 <wire x1="223.95" y1="282.65" x2="223.95" y2="282.4" width="0.1524" layer="91"/>
 </segment>
@@
 </segment>
 </net>
+<net name="N$196" class="0">
+<segment>
+<pinref part="U1" gate="G$1" pin="VCC"/>
+<wire x1="178.71" y1="282.65" x2="223.75" y2="282.65" width="0.1524" layer="91"/>
+</segment>
+</net>

Commit message: fix router
Connections:
- removed net N$196: U1.VCC
- net V_GSM: now also U1.VCC
Changed lines of the file:
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@@
-</segment>
-<segment>
-<wire x1="-54" y1="45.2" x2="-53.6" y2="45.2" width="0.1524" layer="91"/>
-<wire x1="-54" y1="45.15" x2="-54" y2="45.2" width="0.1524" layer="91"/>
-<wire x1="-53.95" y1="45.15" x2="-53.6" y2="45.2" width="0.1524" layer="91"/>
 </segment>
 <segment>
@@
 <pinref part="HUNG" gate="G$1" pin="PA15"/>
 <wire x1="128.53" y1="152.46" x2="128.53" y2="161.26" width="0.1524" layer="91"/>
-</segment>
-</net>
-<net name="N$10" class="0">
-<segment>
-<wire x1="-38.75" y1="45.15" x2="-38.75" y2="45.05" width="0.1524" layer="91"/>
 </segment>
 </net>
@@
 <pinref part="U1" gate="G$1" pin="V_INT"/>
 <wire x1="178.71" y1="277.57" x2="202.98" y2="277.57" width="0.1524" layer="91"/>
-<wire x1="202.98" y1="277.57" x2="202.98" y2="277.36" width="0.1524" layer="91"/>
 <label x="183.92" y="277.82" size="1.778" layer="95"/>
 </segment>
@@
 <pinref part="U1" gate="G$1" pin="V_BCKP"/>
 <wire x1="178.71" y1="280.11" x2="203.57" y2="280.11" width="0.1524" layer="91"/>
-<wire x1="203.57" y1="280.11" x2="203.57" y2="279.99" width="0.1524" layer="91"/>
 <label x="180.4" y="279.99" size="1.778" layer="95"/>
 </segment>
@@
 <net name="V_GSM" class="0">
 <segment>
-<junction x="223.73" y="282.65"/>
-<wire x1="223.73" y1="277.57" x2="223.73" y2="282.65" width="0.1524" layer="91"/>
-<pinref part="C24" gate="G$1" pin="1"/>
-</segment>
-<segment>
 <wire x1="223.8" y1="282.65" x2="233.89" y2="282.65" width="0.1524" layer="91"/>
 <wire x1="233.89" y1="282.65" x2="244.05" y2="282.65" width="0.1524" layer="91"/>
@@
 <wire x1="254.21" y1="282.65" x2="264.37" y2="282.65" width="0.1524" layer="91"/>
 <wire x1="274.53" y1="282.65" x2="287.23" y2="282.65" width="0.1524" layer="91"/>
+<wire x1="223.73" y1="277.57" x2="223.73" y2="282.65" width="0.1524" layer="91"/>
+<junction x="223.73" y="282.65"/>
 <wire x1="233.89" y1="277.57" x2="233.89" y2="282.65" width="0.1524" layer="91"/>
 <junction x="233.89" y="282.65"/>
@@
 <pinref part="C15" gate="G$1" pin="1"/>
 <pinref part="C17" gate="G$1" pin="1"/>
+<pinref part="C24" gate="G$1" pin="1"/>
 <pinref part="V_GSM" gate="G$1" pin="TP"/>
 <pinref part="TVS8" gate="G$1" pin="2"/>
+<pinref part="U1" gate="G$1" pin="VCC"/>
+<wire x1="178.71" y1="282.65" x2="223.75" y2="282.65" width="0.1524" layer="91"/>
 <wire x1="223.8" y1="282.55" x2="223.8" y2="282.65" width="0.1524" layer="91"/>
+<wire x1="223.75" y1="282.65" x2="223.95" y2="282.65" width="0.1524" layer="91"/>
 <wire x1="223.95" y1="282.65" x2="223.95" y2="282.4" width="0.1524" layer="91"/>
 </segment>
@@
 <label x="86.95" y="314.89" size="1.778" layer="95"/>
 </segment>
-<segment>
-<wire x1="203.22" y1="277.57" x2="203.22" y2="277.63" width="0.1524" layer="91"/>
-</segment>
 </net>
 <net name="GSM_EN" class="0">
@@
 </segment>
 </net>
-<net name="N$196" class="0">
-<segment>
-<pinref part="U1" gate="G$1" pin="VCC"/>
-<wire x1="178.71" y1="282.65" x2="223.75" y2="282.65" width="0.1524" layer="91"/>
-</segment>
-</net>

Commit message: fix ERC-Fehler
Connections:
- removed net GSM_PWR_ON1: R14.2, U1.PWR_ON
- removed net N$119: HUNG.PB4
- removed net N$120: HUNG.PB3
- removed net N$44: HUNG.PC4
- removed net N$45: HUNG.PC5
- removed net N$98: HUNG.PD12
- removed net N$99: HUNG.PD11
- removed net VSS: C12.1
- new net GSM_PWR_ON: HUNG.PC5, R14.2, U1.PWR_ON
- net GND: now also C12.1
- net GSM_RESET_N: now also HUNG.PC4
- net PWDN: now also HUNG.PB3
- net RESET: now also HUNG.PB4
Other:
- moved on the sheet: VINT, V_GSM

Commit message: fix power-pins
Other:
- note added: "GSM_MODUL"
Changed lines of the file:
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@@
 <text x="12.4" y="59.45" size="1.778" layer="90">UART</text>
 <text x="21.09" y="304.79" size="2.54" layer="90">Level Shifter</text>
+<text x="159.84" y="293.81" size="5.08" layer="91">GSM_MODUL</text>
 </plain>
 <instances>
@@
 <segment>
 <pinref part="U1" gate="G$1" pin="ANT1"/>
-<wire x1="132.99" y1="272.49" x2="117.88" y2="272.49" width="0.1524" layer="91"/>
+<wire x1="132.99" y1="272.49" x2="109.87" y2="272.49" width="0.1524" layer="91"/>
 <pinref part="ANT2" gate="G$1" pin="SIG"/>
-<wire x1="117.88" y1="272.49" x2="117.88" y2="317.4" width="0.1524" layer="91"/>
-<wire x1="117.88" y1="317.4" x2="137.91" y2="317.4" width="0.1524" layer="91"/>
+<wire x1="109.87" y1="272.49" x2="109.87" y2="317.4" width="0.1524" layer="91"/>
+<wire x1="109.87" y1="317.4" x2="137.91" y2="317.4" width="0.1524" layer="91"/>
 <label x="127.8" y="274.2" size="1.778" layer="95" rot="R180"/>
 </segment>
